File: 5.25 floppy adapter.kicad_pcb (KiCad board)
At the start: 2 copper layers, 44.5 x 25.4 mm, 2 parts

Commit message: PCB layout done
Parts:
- removed Floppy Top: 5.25 Male Edge Connector, FloppyBits:525_male_edge
- removed GOTEK: Pin_Header_Straight_2x17_Pitch2.54mm, Pin_Headers:Pin_Header_Straight_2x17_Pitch2.54mm
- added G1: GOTEK, Pin_Headers:Pin_Header_Straight_2x17_Pitch2.54mm, B.Cu at (170.2, 97.8)
- added N1: 5.25 Floppy Edge Connector, FloppyBits:525_male_edge, F.Cu at (149.9, 82.5)
Routing:
- net (no net): track 553.8 -> 0.00 mm, vias 1 -> 0
- net GND: track 0.00 -> 243.4 mm
- net Net-(G1-Pad10): track 0.00 -> 23.9 mm
- net Net-(G1-Pad14): track 0.00 -> 20.8 mm
- net Net-(G1-Pad8): track 0.00 -> 15.2 mm
- net Net-(G1-Pad32): track 0.00 -> 15.2 mm
- net Net-(G1-Pad30): track 0.00 -> 15.2 mm
- net Net-(G1-Pad28): track 0.00 -> 15.2 mm
- net Net-(G1-Pad26): track 0.00 -> 15.2 mm
- net Net-(G1-Pad24): track 0.00 -> 15.2 mm
- net Net-(G1-Pad22): track 0.00 -> 15.2 mm
- net Net-(G1-Pad20): track 0.00 -> 15.2 mm
- net Net-(G1-Pad18): track 0.00 -> 15.2 mm
- net Net-(G1-Pad12): track 0.00 -> 15.2 mm
Other:
- board outline removed
- board text added: "PC-8801mkII floppy adapter v1.0"
- board text added: "THIS SIDE DOWN"
- board text removed: "1"
- board text removed: "2"
- board text removed: "33"
- board text removed: "34"
- board text removed: "5.25" -> 3.5" floppy (PC8801mkII)"
- board text removed: "GROUND SIDE"

Commit message: Fully routed PCB
Routing:
- net GND: track 243.4 -> 255.5 mm, vias 0 -> 1
Other:
- board outline added: 48.3 x 26 mm
Changed lines of the file:
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@@
   (general
     (thickness 1.6)
-    (drawings 3)
-    (tracks 53)
+    (drawings 11)
+    (tracks 55)
     (zones 0)
     (modules 2)
@@
     )
   )
+  (gr_line (start 128.27 90.17) (end 128.27 74.295) (layer Edge.Cuts) (width 0.15))
+  (gr_line (start 125.73 92.71) (end 128.27 90.17) (layer Edge.Cuts) (width 0.15))
+  (gr_line (start 125.73 100.33) (end 125.73 92.71) (layer Edge.Cuts) (width 0.15))
+  (gr_line (start 173.99 100.33) (end 125.73 100.33) (layer Edge.Cuts) (width 0.15))
+  (gr_line (start 173.99 94.615) (end 173.99 100.33) (layer Edge.Cuts) (width 0.15))
+  (gr_line (start 171.45 92.075) (end 173.99 94.615) (layer Edge.Cuts) (width 0.15))
+  (gr_line (start 171.45 74.295) (end 171.45 92.075) (layer Edge.Cuts) (width 0.15))
+  (gr_line (start 128.27 74.295) (end 171.45 74.295) (layer Edge.Cuts) (width 0.15))
   (gr_text www.leadedsolder.com (at 149.86 91.44) (layer B.SilkS)
     (effects (font (size 1.5 1.5) (thickness 0.3)) (justify mirror))
@@
   )
   (segment (start 170.18 97.79) (end 129.54 97.79) (width 0.25) (layer B.Cu) (net 2))
-  (segment (start 128.364999 96.614999) (end 128.690001 96.940001) (width 0.25) (layer B.Cu) (net 2))
-  (segment (start 128.690001 96.940001) (end 129.54 97.79) (width 0.25) (layer B.Cu) (net 2))
-  (segment (start 129.54 85.635) (end 128.364999 86.810001) (width 0.25) (layer B.Cu) (net 2))
   (segment (start 129.54 80.01) (end 129.54 85.635) (width 0.25) (layer B.Cu) (net 2))
   (segment (start 170.18 80.01) (end 170.18 88.9) (width 0.25) (layer B.Cu) (net 2))
-  (segment (start 128.364999 88.9) (end 128.364999 96.614999) (width 0.25) (layer B.Cu) (net 2))
-  (segment (start 128.364999 86.810001) (end 128.364999 88.9) (width 0.25) (layer B.Cu) (net 2))
   (segment (start 132.08 80.01) (end 132.08 88.9) (width 0.25) (layer B.Cu) (net 2))
-  (segment (start 132.08 88.9) (end 128.364999 88.9) (width 0.25) (layer B.Cu) (net 2))
   (segment (start 134.62 88.9) (end 132.08 88.9) (width 0.25) (layer B.Cu) (net 2))
   (segment (start 134.62 80.01) (end 134.62 88.9) (width 0.25) (layer B.Cu) (net 2))
@@
   (segment (start 167.64 88.9) (end 162.56 88.9) (width 0.25) (layer B.Cu) (net 2))
   (segment (start 170.18 88.9) (end 167.64 88.9) (width 0.25) (layer B.Cu) (net 2))
+  (segment (start 129.54 92.075) (end 129.54 86.995) (width 0.25) (layer B.Cu) (net 2))
+  (segment (start 127.635 93.98) (end 129.54 92.075) (width 0.25) (layer B.Cu) (net 2))
+  (segment (start 127.635 95.885) (end 127.635 93.98) (width 0.25) (layer B.Cu) (net 2))
+  (segment (start 129.54 97.79) (end 127.635 95.885) (width 0.25) (layer B.Cu) (net 2))
+  (segment (start 132.08 88.9) (end 129.54 88.9) (width 0.25) (layer B.Cu) (net 2))
+  (segment (start 129.54 86.995) (end 129.54 80.01) (width 0.25) (layer B.Cu) (net 2))
+  (via (at 129.54 86.995) (size 0.8) (drill 0.4) (layers F.Cu B.Cu) (net 2))
+  (segment (start 129.54 80.01) (end 129.54 86.995) (width 0.25) (layer F.Cu) (net 2))
   (segment (start 132.08 95.25) (end 132.08 80.01) (width 0.25) (layer F.Cu) (net 3))
   (segment (start 134.62 95.25) (end 134.62 80.01) (width 0.25) (layer F.Cu) (net 4))
