File: 5.25 floppy adapter.kicad_pcb (KiCad board)
At the start: 2 copper layers, 44.2 x 21.3 mm, 2 parts

Commit message: Big nasty slot
Routing:
- net Net-(G1-Pad24): track 14.7 -> 18.4 mm
Other:
- outline, holes or cut-outs redrawn
- board text added: "edge-connector floppy adapter v2.3"
- board text removed: "edge-connector floppy adapter v2.2"
Changed lines of the file:
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@@
   (general
     (thickness 1.6)
-    (drawings 17)
-    (tracks 128)
+    (drawings 21)
+    (tracks 129)
     (zones 0)
     (modules 2)
@@
       (net 13 GND) (clearance 0.375))
   )
-  (gr_line (start 155.956 78.232) (end 199.009 78.232) (layer Edge.Cuts) (width 0.15))
+  (gr_line (start 193.929 78.232) (end 155.956 78.232) (layer Edge.Cuts) (width 0.15))
+  (gr_line (start 194.564 90.678) (end 193.929 90.678) (layer Edge.Cuts) (width 0.15))
+  (gr_line (start 194.564 78.232) (end 199.009 78.232) (layer Edge.Cuts) (width 0.15))
+  (gr_line (start 193.929 90.678) (end 193.929 78.232) (layer Edge.Cuts) (width 0.15))
+  (gr_line (start 194.564 78.232) (end 194.564 90.678) (layer Edge.Cuts) (width 0.15))
   (gr_line (start 155.448 78.867) (end 155.956 78.232) (layer Edge.Cuts) (width 0.15))
   (gr_line (start 199.644 78.867) (end 199.009 78.232) (layer Edge.Cuts) (width 0.15))
@@
     (effects (font (size 0.85 0.85) (thickness 0.2125)))
   )
-  (gr_text "edge-connector floppy adapter v2.2" (at 170.942 92.71) (layer F.SilkS)
+  (gr_text "edge-connector floppy adapter v2.3" (at 170.942 92.71) (layer F.SilkS)
     (effects (font (size 0.75 0.75) (thickness 0.1875)))
   )
@@
   (segment (start 172.61 84.115) (end 172.61 93.582) (width 0.25) (layer F.Cu) (net 7))
   (segment (start 169.316401 96.926401) (end 170.18 97.79) (width 0.25) (layer F.Cu) (net 8))
-  (segment (start 168.828601 89.836399) (end 168.828601 96.438601) (width 0.25) (layer F.Cu) (net 8))
-  (segment (start 170.07 88.595) (end 168.828601 89.836399) (width 0.25) (layer F.Cu) (net 8))
   (segment (start 168.828601 96.438601) (end 169.316401 96.926401) (width 0.25) (layer F.Cu) (net 8))
   (segment (start 170.07 84.115) (end 170.07 88.595) (width 0.25) (layer F.Cu) (net 8))
+  (segment (start 168.828601 91.812399) (end 168.828601 96.438601) (width 0.25) (layer F.Cu) (net 8))
+  (segment (start 170.053 90.588) (end 168.828601 91.812399) (width 0.25) (layer F.Cu) (net 8))
+  (segment (start 170.053 84.963) (end 170.053 90.588) (width 0.25) (layer F.Cu) (net 8))
   (segment (start 166.776401 96.926401) (end 167.64 97.79) (width 0.25) (layer F.Cu) (net 9))
   (segment (start 166.288601 90.981399) (end 166.288601 96.438601) (width 0.25) (layer F.Cu) (net 9))
