File: 5.25 floppy adapter.sch (KiCad schematic (older format))
At the start: 2 parts

Commit message: added an actual IDC connector and flipped the board around so it will actually work this time
Parts:
- G1: footprint Pin_Headers:Pin_Header_Straight_2x17_Pitch2.54mm -> Connector_IDC:IDC-Header_2x17_P2.54mm_Horizontal
Changed lines of the file:
@@
 F 0 "G1" H 5475 5017 50  0000 C CNN
 F 1 "GOTEK" H 5475 4926 50  0000 C CNN
-F 2 "Pin_Headers:Pin_Header_Straight_2x17_Pitch2.54mm" H 5425 4000 50  0001 C CNN
+F 2 "Connector_IDC:IDC-Header_2x17_P2.54mm_Horizontal" H 5425 4000 50  0001 C CNN
 F 3 "~" H 5425 4000 50  0001 C CNN
 	1    5425 4000

Commit message: Straight-through version
Connections:
- wire segments 90 -> 88
Changed lines of the file:
@@
 	1    0    0    -1
 $EndComp
-Wire Wire Line
-	8200 4800 6875 4800
-Wire Wire Line
-	6875 4800 6875 5075
 $Comp
 L Connector_Generic:Conn_02x17_Odd_Even G1
@@
 $EndComp
 Wire Wire Line
-	8200 3500 5725 3500
-Wire Wire Line
-	8200 3900 6500 3900
-Wire Wire Line
-	5725 3600 6500 3600
-Wire Wire Line
-	6500 3600 6500 3900
-Connection ~ 6500 3900
-Wire Wire Line
-	6500 3900 5725 3900
-Wire Wire Line
-	8200 3700 5725 3700
-Wire Wire Line
-	8200 3600 7300 3600
-Wire Wire Line
-	7300 3600 7300 3800
-Wire Wire Line
-	7300 3800 5725 3800
-Wire Wire Line
-	5725 4000 8200 4000
-Wire Wire Line
-	8200 4100 5725 4100
-Wire Wire Line
-	5725 4200 8200 4200
-Wire Wire Line
-	8200 4300 5725 4300
-Wire Wire Line
-	5725 4400 8200 4400
-Wire Wire Line
-	8200 4500 5725 4500
-Wire Wire Line
-	5725 4600 8200 4600
-Wire Wire Line
-	8200 4700 5725 4700
-Wire Wire Line
 	8700 3200 9025 3200
 Wire Wire Line
@@
 Wire Wire Line
 	5025 4800 5025 5075
+Wire Wire Line
+	8200 4800 5725 4800
+Wire Wire Line
+	5725 4700 8200 4700
+Wire Wire Line
+	8200 4600 5725 4600
+Wire Wire Line
+	5725 4500 8200 4500
+Wire Wire Line
+	8200 4400 5725 4400
+Wire Wire Line
+	5725 4300 8200 4300
+Wire Wire Line
+	8200 4200 5725 4200
+Wire Wire Line
+	5725 4100 8200 4100
+Wire Wire Line
+	8200 4000 5725 4000
+Wire Wire Line
+	5725 3900 8200 3900
+Wire Wire Line
+	8200 3800 5725 3800
+Wire Wire Line
+	5725 3700 8200 3700
+Wire Wire Line
+	8200 3600 5725 3600
+Wire Wire Line
+	5725 3500 8200 3500
+Wire Wire Line
+	8200 3400 5725 3400
+Wire Wire Line
+	5725 3300 8200 3300
+Wire Wire Line
+	8200 3200 5725 3200
 $EndSCHEMATC

Commit message: Label the schematic
Connections:
- net labels added: Direction, DriveSelect0, DriveSelect1, DriveSelect2, DriveSelect3, Index, MotorOn, READY, ReadData, SideSelect, Step, Track0, WriteData, WriteGate, WriteProtect
Changed lines of the file:
@@
 EESchema Schematic File Version 4
+LIBS:5.25 floppy adapter-cache
 EELAYER 26 0
 EELAYER END
@@
 Wire Wire Line
 	8200 3200 5725 3200
+Text Label 8200 4800 2    50   ~ 0
+READY
+Text Label 5725 4800 0    50   ~ 0
+READY
+Text Label 5725 3400 0    50   ~ 0
+DriveSelect3
+Text Label 8200 3400 2    50   ~ 0
+DriveSelect3
+Text Label 8200 3500 2    50   ~ 0
+Index
+Text Label 5725 3500 0    50   ~ 0
+Index
+Text Label 5725 3600 0    50   ~ 0
+DriveSelect0
+Text Label 8200 3600 2    50   ~ 0
+DriveSelect0
+Text Label 8200 3700 2    50   ~ 0
+DriveSelect1
+Text Label 5725 3700 0    50   ~ 0
+DriveSelect1
+Text Label 5725 3800 0    50   ~ 0
+DriveSelect2
+Text Label 5725 3900 0    50   ~ 0
+MotorOn
+Text Label 5725 4000 0    50   ~ 0
+Direction
+Text Label 5725 4100 0    50   ~ 0
+Step
+Text Label 5725 4200 0    50   ~ 0
+WriteData
+Text Label 5725 4300 0    50   ~ 0
+WriteGate
+Text Label 5725 4400 0    50   ~ 0
+Track0
+Text Label 5725 4500 0    50   ~ 0
+WriteProtect
+Text Label 5725 4600 0    50   ~ 0
+ReadData
+Text Label 5725 4700 0    50   ~ 0
+SideSelect
+Text Label 8200 3800 2    50   ~ 0
+DriveSelect2
+Text Label 8175 3900 2    50   ~ 0
+MotorOn
+Text Label 8200 4000 2    50   ~ 0
+Direction
+Text Label 8200 4100 2    50   ~ 0
+Step
+Text Label 8200 4200 2    50   ~ 0
+WriteData
+Text Label 8200 4300 2    50   ~ 0
+WriteGate
+Text Label 8200 4400 2    50   ~ 0
+Track0
+Text Label 8200 4500 2    50   ~ 0
+WriteProtect
+Text Label 8200 4600 2    50   ~ 0
+ReadData
+Text Label 8200 4700 2    50   ~ 0
+SideSelect
 $EndSCHEMATC

Commit message: Use the straight-through Shugart variant (#1)
* Straight-through variant

* Gerber plot options

* Fewer corner departures from pads
Connections:
- net labels removed: Direction, DriveSelect0, DriveSelect1, DriveSelect2, DriveSelect3, Index, MotorOn, READY, ReadData, SideSelect, Step, Track0, WriteData, WriteGate, WriteProtect
Changed lines of the file:
@@
 Wire Wire Line
 	8200 3200 5725 3200
-Text Label 8200 4800 2    50   ~ 0
-READY
-Text Label 5725 4800 0    50   ~ 0
-READY
-Text Label 5725 3400 0    50   ~ 0
-DriveSelect3
-Text Label 8200 3400 2    50   ~ 0
-DriveSelect3
-Text Label 8200 3500 2    50   ~ 0
-Index
-Text Label 5725 3500 0    50   ~ 0
-Index
-Text Label 5725 3600 0    50   ~ 0
-DriveSelect0
-Text Label 8200 3600 2    50   ~ 0
-DriveSelect0
-Text Label 8200 3700 2    50   ~ 0
-DriveSelect1
-Text Label 5725 3700 0    50   ~ 0
-DriveSelect1
-Text Label 5725 3800 0    50   ~ 0
-DriveSelect2
-Text Label 5725 3900 0    50   ~ 0
-MotorOn
-Text Label 5725 4000 0    50   ~ 0
-Direction
-Text Label 5725 4100 0    50   ~ 0
-Step
-Text Label 5725 4200 0    50   ~ 0
-WriteData
-Text Label 5725 4300 0    50   ~ 0
-WriteGate
-Text Label 5725 4400 0    50   ~ 0
-Track0
-Text Label 5725 4500 0    50   ~ 0
-WriteProtect
-Text Label 5725 4600 0    50   ~ 0
-ReadData
-Text Label 5725 4700 0    50   ~ 0
-SideSelect
-Text Label 8200 3800 2    50   ~ 0
-DriveSelect2
-Text Label 8175 3900 2    50   ~ 0
-MotorOn
-Text Label 8200 4000 2    50   ~ 0
-Direction
-Text Label 8200 4100 2    50   ~ 0
-Step
-Text Label 8200 4200 2    50   ~ 0
-WriteData
-Text Label 8200 4300 2    50   ~ 0
-WriteGate
-Text Label 8200 4400 2    50   ~ 0
-Track0
-Text Label 8200 4500 2    50   ~ 0
-WriteProtect
-Text Label 8200 4600 2    50   ~ 0
-ReadData
-Text Label 8200 4700 2    50   ~ 0
-SideSelect
 $EndSCHEMATC
